Commit message: update

File: control_robotarm/urdf/model.URDF (robot description, URDF)
Before this commit: robot RobotArm_latest_v4, 8 links, 7 joints
Links:
- link 1axisUnit_V2_v1:1: geometry collision mesh filename=package:../meshes/1axisUnit_V2_v1.stl scale=1.0 1.0 1.0; visual mesh filename=package:../meshes/1axisUnit_V2_v1.stl scale=1.0 1.0 1.0
- link 2axisUnit_V2_v1:1: geometry collision mesh filename=package:../meshes/2axisUnit_V2_v1.stl scale=1.0 1.0 1.0; visual mesh filename=package:../meshes/2axisUnit_V2_v1.stl scale=1.0 1.0 1.0
- link 3axisUnit_V3_v1:1: geometry collision mesh filename=package:../meshes/3axisUnit_V3_v1.stl scale=1.0 1.0 1.0; visual mesh filename=package:../meshes/3axisUnit_V3_v1.stl scale=1.0 1.0 1.0
