Commit message: mkdir todoroki_arm

File: control_robotarm/todoroki_arm/todoroki_robotarm.URDF (robot description, URDF)
Before this commit: robot RobotArm_latest_v4, 8 links, 7 joints
Joints:
- joint rev0: limit lower=-3.15 upper=3.15 effort=0 velocity=0 -> (none)
- joint rev1: limit lower=-3.15 upper=3.15 effort=0 velocity=0 -> (none); origin xyz=-0.026 0 0.1 rpy=0 0 0 -> xyz=-0.0 0 0.1 rpy=0 0 0
- joint rev2: limit lower=-3.15 upper=3.15 effort=0 velocity=0 -> (none)
- joint rev3: limit lower=-3.15 upper=3.15 effort=0 velocity=0 -> (none)
- joint rev4: limit lower=-3.15 upper=3.15 effort=0 velocity=0 -> (none)
- joint rev5: limit lower=-3.15 upper=3.15 effort=0 velocity=0 -> (none)
- joint rev6: limit lower=-3.15 upper=3.15 effort=0 velocity=0 -> (none)
