Commit message: update

File: control_robotarm/todoroki_arm/todoroki_robotarm.urdf (robot description, URDF)
Before this commit: robot RobotArm_latest_v4, 8 links, 7 joints
Joints:
- removed joint rev5
- removed joint rev6
- joint rev2: origin xyz=0.04550000000005672 0.030999999999995993 0.29650000000128046 rpy=0 0 0 -> xyz=0 0 0.29650000000128046 rpy=0 0 0
- joint rev3: origin xyz=0 -0.030 0.30 rpy=0 0 0 -> xyz=0 -0.0 0.30 rpy=0 0 0
- joint rev4: origin xyz=-0.01999999091727354 0 0.06149999999619804 rpy=0 0 0 -> xyz=0 0 0.06149999999619804 rpy=0 0 0

Commit message: update

File: control_robotarm/todoroki_arm/todoroki_robotarm.urdf (robot description, URDF)
Before this commit: robot RobotArm_latest_v4, 8 links, 5 joints
Joints:
- joint rev2: axis -1.0 0 0 -> 1.0 0 0
