Commit message: update

File: old_ver/todoroki_robotarm.urdf (robot description, URDF)
Before this commit: robot RobotArm_latest_v4, 8 links, 5 joints
Joints:
- joint rev1: axis -1.0 0 0 -> 1.0 0 0

Commit message: update

File: old_ver/todoroki_robotarm.urdf (robot description, URDF)
Before this commit: robot RobotArm_latest_v4, 8 links, 5 joints
Joints:
- joint rev1: axis 1.0 0 0 -> -1.0 0 0

Commit message: update

File: old_ver/todoroki_robotarm.urdf (robot description, URDF)
Before this commit: robot RobotArm_latest_v4, 8 links, 5 joints
Joints:
- joint rev4: origin xyz=0 0 0.1240 rpy=0 0 0 -> xyz=0 0 0.340 rpy=0 0 0
